File: electronics/project.kicad_pcb (KiCad board)
At the start: 2 copper layers, 31.8 x 58.4 mm, 32 parts, among them P1 TRINKET_LEFT, P2 TRINKET_RIGHT, P3 RIGHT_STEPPER, P4 LEFT_STEPPER, P5 BATT1, P6 BATT2, P7 SERVO, P8 A5 - A1, P9 CONN_01X01, Q1 OPTO_NPN, Q2 OPTO_NPN, SW1 SPST, SW2 SW_PUSH, U1 ULN2803

Commit message: Update PCB link and BOM
Parts:
- C1: footprint Capacitors_ThroughHole:C_Radial_D7.5_L11.2_P2.5 -> footprints:C_Radial_D7.5_L11.2_P2.5
- C2: footprint Capacitors_ThroughHole:C_Radial_D5_L11_P2.5 -> footprints:C_Radial_D5_L11_P2.5
- C3: footprint Capacitors_ThroughHole:C_Disc_D3_P2.5 -> footprints:C_Disc_D3_P2.5
- D2, D3, D4, D5: footprint LEDs:LED-3MM -> footprints:LED-3MM
- P1, P2: footprint Pin_Headers:Pin_Header_Straight_1x12 -> footprints:Pin_Header_Straight_1x12
- P3, P4: footprint library:JST_B5B-XH-A -> footprints:JST_B5B-XH-A
- P5, P6: footprint Terminal_Blocks:TerminalBlock_Pheonix_PT-3.5mm_2pol -> footprints:TerminalBlock_Pheonix_PT-3.5mm_2pol
- P7, P8: footprint Pin_Headers:Pin_Header_Straight_1x03 -> footprints:Pin_Header_Straight_1x03
- Q1, Q2: footprint myFootPrints:PHOTOTRANS -> footprints:PHOTOTRANS
- R2, R4, R5, R6, R7: footprint myFootPrints:Resistor_Horz -> footprints:Resistor_Horz
- R3: value 300 -> 330; footprint myFootPrints:Resistor_Horz -> footprints:Resistor_Horz
- SW1: footprint myFootPrints:SW_Micro_SPST -> footprints:SW_Micro_SPST
- SW2: footprint myFootPrints:SW_PUSH_SMALL -> footprints:SW_PUSH_SMALL
- U1: footprint Housings_DIP:DIP-18_W7.62mm -> footprints:DIP-18_W7.62mm
Connections:
- P1 pad 6: (no net) -> /AREF
- P2 pad 10: /D2 -> /D1
- P2 pad 11: /D1 -> /D0
- P2 pad 12: (no net) -> /RST
- P2 pad 3: (no net) -> /VBUS
- R4 pad 1: /D2 -> /D1
- R5 pad 1: /D1 -> /D0
Routing:
- net /D2: track 28.1 -> 0.00 mm
- net /D0: track 0.00 -> 19.2 mm
- net /D1: track 19.2 -> 28.1 mm
