File: electronics/project.sch (KiCad schematic (older format))
At the start: 26 parts, among them P1 TRINKET_LEFT, P2 TRINKET_RIGHT, P3 RIGHT_STEPPER, P4 LEFT_STEPPER, P5 BATT1, P6 BATT2, P7 SERVO, P8 A5 - A1, Q1 OPTO_NPN, Q2 OPTO_NPN, SW1 SPST, SW2 SW_PUSH, U1 ULN2803

Commit message: Update PCB link and BOM
Parts:
- C1: footprint Capacitors_ThroughHole:C_Radial_D7.5_L11.2_P2.5 -> footprints:C_Radial_D7.5_L11.2_P2.5
- C2: footprint Capacitors_ThroughHole:C_Radial_D5_L11_P2.5 -> footprints:C_Radial_D5_L11_P2.5
- C3: footprint Capacitors_ThroughHole:C_Disc_D3_P2.5 -> footprints:C_Disc_D3_P2.5
- D2, D3, D4, D5: footprint LEDs:LED-3MM -> footprints:LED-3MM; symbol LED -> LED-RESCUE-base
- P1, P2: footprint Pin_Headers:Pin_Header_Straight_1x12 -> footprints:Pin_Header_Straight_1x12
- P3, P4: footprint Terminal_Blocks:TerminalBlock_Pheonix_MPT-2.54mm_2pol -> footprints:JST_B5B-XH-A
- P5, P6: footprint Terminal_Blocks:TerminalBlock_Pheonix_MPT-2.54mm_2pol -> footprints:TerminalBlock_Pheonix_PT-3.5mm_2pol
- P7, P8: footprint Pin_Headers:Pin_Header_Straight_1x03 -> footprints:Pin_Header_Straight_1x03
- Q1, Q2: footprint myFootPrints:PHOTOTRANS -> footprints:PHOTOTRANS
- R2, R3, R4, R5, R6, R7: footprint myFootPrints:Resistor_Horz -> footprints:Resistor_Horz
- SW1: footprint myFootPrints:SW_Micro_SPST -> footprints:SW_Micro_SPST
- SW2: footprint myFootPrints:SW_PUSH_SMALL -> footprints:SW_PUSH_SMALL
- U1: footprint Housings_DIP:DIP-18_W7.62mm -> footprints:DIP-18_W7.62mm
Changed lines of the file:
@@
 EESchema Schematic File Version 2
-LIBS:base-rescue
+LIBS:project
 LIBS:power
 LIBS:device
@@
 LIBS:contrib
 LIBS:valves
-LIBS:MMA8452Q
-LIBS:w_analog
-LIBS:base-cache
+LIBS:project-cache
 EELAYER 25 0
 EELAYER END
@@
 F 0 "P1" H 4800 4050 50  0000 C CNN
 F 1 "TRINKET_LEFT" V 4900 3400 50  0000 C CNN
-F 2 "Pin_Headers:Pin_Header_Straight_1x12" H 4800 3400 50  0001 C CNN
+F 2 "footprints:Pin_Header_Straight_1x12" H 4800 3400 50  0001 C CNN
 F 3 "" H 4800 3400 50  0000 C CNN
 	1    4800 3400
@@
 F 0 "P2" H 5450 4050 50  0000 C CNN
 F 1 "TRINKET_RIGHT" V 5550 3400 50  0000 C CNN
-F 2 "Pin_Headers:Pin_Header_Straight_1x12" H 5450 3400 50  0001 C CNN
+F 2 "footprints:Pin_Header_Straight_1x12" H 5450 3400 50  0001 C CNN
 F 3 "" H 5450 3400 50  0000 C CNN
 	1    5450 3400
@@
 F 0 "U1" H 8250 4100 60  0000 C CNN
 F 1 "ULN2803" H 8350 4000 60  0000 C CNN
-F 2 "Housings_DIP:DIP-18_W7.62mm" H 8100 3550 60  0001 C CNN
+F 2 "footprints:DIP-18_W7.62mm" H 8100 3550 60  0001 C CNN
 F 3 "" H 8100 3550 60  0000 C CNN
 	1    8100 3550
@@
 F 0 "P3" H 9300 3450 50  0000 C CNN
 F 1 "RIGHT_STEPPER" V 9400 3150 50  0000 C CNN
-F 2 "Terminal_Blocks:TerminalBlock_Pheonix_MPT-2.54mm_2pol" H 9300 3150 50  0001 C CNN
+F 2 "footprints:JST_B5B-XH-A" H 9300 3150 50  0001 C CNN
 F 3 "" H 9300 3150 50  0000 C CNN
 	1    9300 3150
@@
 F 0 "P4" H 9300 4100 50  0000 C CNN
 F 1 "LEFT_STEPPER" V 9400 3800 50  0000 C CNN
-F 2 "Terminal_Blocks:TerminalBlock_Pheonix_MPT-2.54mm_2pol" H 9300 3800 50  0001 C CNN
+F 2 "footprints:JST_B5B-XH-A" H 9300 3800 50  0001 C CNN
 F 3 "" H 9300 3800 50  0000 C CNN
 	1    9300 3800
@@
 F 0 "P5" H 6500 2050 50  0000 C CNN
 F 1 "BATT1" V 6600 1900 50  0000 C CNN
-F 2 "Terminal_Blocks:TerminalBlock_Pheonix_MPT-2.54mm_2pol" H 6500 1900 50  0001 C CNN
+F 2 "footprints:TerminalBlock_Pheonix_PT-3.5mm_2pol" H 6500 1900 50  0001 C CNN
 F 3 "" H 6500 1900 50  0000 C CNN
 	1    6500 1900
@@
 F 0 "P6" H 6800 2050 50  0000 C CNN
 F 1 "BATT2" V 6900 1900 50  0000 C CNN
-F 2 "Terminal_Blocks:TerminalBlock_Pheonix_MPT-2.54mm_2pol" H 6800 1900 50  0001 C CNN
+F 2 "footprints:TerminalBlock_Pheonix_PT-3.5mm_2pol" H 6800 1900 50  0001 C CNN
 F 3 "" H 6800 1900 50  0000 C CNN
 	1    6800 1900
@@
 F 0 "SW1" H 7350 2200 50  0000 C CNN
 F 1 "SPST" H 7350 2000 50  0000 C CNN
-F 2 "myFootPrints:SW_Micro_SPST" H 7350 2100 50  0001 C CNN
+F 2 "footprints:SW_Micro_SPST" H 7350 2100 50  0001 C CNN
 F 3 "" H 7350 2100 50  0000 C CNN
 	1    7350 2100
@@
 F 0 "P7" H 8800 2400 50  0000 C CNN
 F 1 "SERVO" V 8900 2200 50  0000 C CNN
-F 2 "Pin_Headers:Pin_Header_Straight_1x03" H 8800 2200 50  0001 C CNN
+F 2 "footprints:Pin_Header_Straight_1x03" H 8800 2200 50  0001 C CNN
 F 3 "" H 8800 2200 50  0000 C CNN
 	1    8800 2200
@@
 F 0 "C1" H 6725 3100 50  0000 L CNN
 F 1 "100uF" H 6600 3200 50  0000 L CNN
-F 2 "Capacitors_ThroughHole:C_Radial_D7.5_L11.2_P2.5" H 6738 2850 50  0001 C CNN
+F 2 "footprints:C_Radial_D7.5_L11.2_P2.5" H 6738 2850 50  0001 C CNN
 F 3 "" H 6700 3000 50  0000 C CNN
 	1    6700 3000
@@
 F 0 "C2" H 6975 3100 50  0000 L CNN
 F 1 "10uF" H 6900 3200 50  0000 L CNN
-F 2 "Capacitors_ThroughHole:C_Radial_D5_L11_P2.5" H 6988 2850 50  0001 C CNN
+F 2 "footprints:C_Radial_D5_L11_P2.5" H 6988 2850 50  0001 C CNN
 F 3 "" H 6950 3000 50  0000 C CNN
 	1    6950 3000
@@
 F 0 "C3" H 7175 3100 50  0000 L CNN
 F 1 "1uF" H 7150 3200 50  0000 L CNN
-F 2 "Capacitors_ThroughHole:C_Disc_D3_P2.5" H 7188 2850 50  0001 C CNN
+F 2 "footprints:C_Disc_D3_P2.5" H 7188 2850 50  0001 C CNN
 F 3 "" H 7150 3000 50  0000 C CNN
 	1    7150 3000
@@
 F 0 "P8" H 3350 6300 50  0000 C CNN
 F 1 "A5 - A1" V 3450 6100 50  0000 C CNN
-F 2 "Pin_Headers:Pin_Header_Straight_1x03" H 3350 6100 50  0001 C CNN
+F 2 "footprints:Pin_Header_Straight_1x03" H 3350 6100 50  0001 C CNN
 F 3 "" H 3350 6100 50  0000 C CNN
 	1    3350 6100
@@
 F 0 "Q1" H 6550 6250 50  0000 L CNN
 F 1 "OPTO_NPN" V 6450 5800 50  0000 L CNN
-F 2 "myFootPrints:PHOTOTRANS" H 6600 6000 50  0001 C CNN
+F 2 "footprints:PHOTOTRANS" H 6600 6000 50  0001 C CNN
 F 3 "" H 6600 6000 50  0000 C CNN
 	1    6600 6000
@@
 F 0 "Q2" H 8000 6250 50  0000 L CNN
 F 1 "OPTO_NPN" V 8150 5850 50  0000 L CNN
-F 2 "myFootPrints:PHOTOTRANS" H 8000 6000 50  0001 C CNN
+F 2 "footprints:PHOTOTRANS" H 8000 6000 50  0001 C CNN
 F 3 "" H 8000 6000 50  0000 C CNN
 	1    8000 6000
@@
 $EndComp
 $Comp
-L LED D3
+L LED-RESCUE-base D3
 U 1 1 59FA74B3
 P 7150 6000
 F 0 "D3" H 7150 6100 50  0000 C CNN
 F 1 "LED" H 7150 5900 50  0000 C CNN
-F 2 "LEDs:LED-3MM" H 7150 6000 50  0001 C CNN
+F 2 "footprints:LED-3MM" H 7150 6000 50  0001 C CNN
 F 3 "" H 7150 6000 50  0000 C CNN
 	1    7150 6000
@@
 $EndComp
 $Comp
-L LED D5
+L LED-RESCUE-base D5
 U 1 1 59FA75F8
 P 6900 6000
 F 0 "D5" H 6900 6100 50  0000 C CNN
 F 1 "IR LED" H 6900 5900 50  0000 C CNN
-F 2 "LEDs:LED-3MM" H 6900 6000 50  0001 C CNN
+F 2 "footprints:LED-3MM" H 6900 6000 50  0001 C CNN
 F 3 "" H 6900 6000 50  0000 C CNN
 	1    6900 6000
@@
 $EndComp
 $Comp
-L LED D4
+L LED-RESCUE-base D4
 U 1 1 59FA764A
 P 7550 6000
 F 0 "D4" H 7550 6100 50  0000 C CNN
 F 1 "LED" H 7550 5900 50  0000 C CNN
-F 2 "LEDs:LED-3MM" H 7550 6000 50  0001 C CNN
+F 2 "footprints:LED-3MM" H 7550 6000 50  0001 C CNN
 F 3 "" H 7550 6000 50  0000 C CNN
 	1    7550 6000
@@
 $EndComp
 $Comp
-L LED D2
+L LED-RESCUE-base D2
 U 1 1 59FA769F
 P 7800 6000
 F 0 "D2" H 7800 6100 50  0000 C CNN
 F 1 "IR_LED" H 7800 5900 50  0000 C CNN
-F 2 "LEDs:LED-3MM" H 7800 6000 50  0001 C CNN
+F 2 "footprints:LED-3MM" H 7800 6000 50  0001 C CNN
 F 3 "" H 7800 6000 50  0000 C CNN
 	1    7800 6000
@@
 F 0 "R3" V 7230 5650 50  0000 C CNN
 F 1 "330" V 7150 5650 50  0000 C CNN
-F 2 "myFootPrints:Resistor_Horz" V 7080 5650 50  0001 C CNN
+F 2 "footprints:Resistor_Horz" V 7080 5650 50  0001 C CNN
 F 3 "" H 7150 5650 50  0000 C CNN
 	1    7150 5650
@@
 F 0 "R4" V 7630 5650 50  0000 C CNN
 F 1 "330" V 7550 5650 50  0000 C CNN
-F 2 "myFootPrints:Resistor_Horz" V 7480 5650 50  0001 C CNN
+F 2 "footprints:Resistor_Horz" V 7480 5650 50  0001 C CNN
 F 3 "" H 7550 5650 50  0000 C CNN
 	1    7550 5650
@@
 F 0 "R2" V 7880 5650 50  0000 C CNN
 F 1 "100" V 7800 5650 50  0000 C CNN
-F 2 "myFootPrints:Resistor_Horz" V 7730 5650 50  0001 C CNN
+F 2 "footprints:Resistor_Horz" V 7730 5650 50  0001 C CNN
 F 3 "" H 7800 5650 50  0000 C CNN
 	1    7800 5650
@@
 F 0 "R5" V 6980 5650 50  0000 C CNN
 F 1 "100" V 6900 5650 50  0000 C CNN
-F 2 "myFootPrints:Resistor_Horz" V 6830 5650 50  0001 C CNN
+F 2 "footprints:Resistor_Horz" V 6830 5650 50  0001 C CNN
 F 3 "" H 6900 5650 50  0000 C CNN
 	1    6900 5650
@@
 F 0 "R6" V 5480 4800 50  0000 C CNN
 F 1 "10K" V 5400 4800 50  0000 C CNN
-F 2 "myFootPrints:Resistor_Horz" V 5330 4800 50  0001 C CNN
+F 2 "footprints:Resistor_Horz" V 5330 4800 50  0001 C CNN
 F 3 "" H 5400 4800 50  0000 C CNN
 	1    5400 4800
@@
 F 0 "R7" V 5280 4800 50  0000 C CNN
 F 1 "10K" V 5200 4800 50  0000 C CNN
-F 2 "myFootPrints:Resistor_Horz" V 5130 4800 50  0001 C CNN
+F 2 "footprints:Resistor_Horz" V 5130 4800 50  0001 C CNN
 F 3 "" H 5200 4800 50  0000 C CNN
 	1    5200 4800
@@
 Connection ~ 5400 5100
 Wire Wire Line
-	6150 4400 6150 3150
-Wire Wire Line
-	5200 4400 6150 4400
+	6150 3150 6150 4400
+Wire Wire Line
+	6150 4400 5200 4400
 Wire Wire Line
 	5200 4400 5200 4650
@@
 F 0 "SW2" H 3900 5560 50  0000 C CNN
 F 1 "SW_PUSH" H 3750 5370 50  0000 C CNN
-F 2 "myFootPrints:SW_PUSH_SMALL" H 3750 5450 50  0001 C CNN
+F 2 "footprints:SW_PUSH_SMALL" H 3750 5450 50  0001 C CNN
 F 3 "" H 3750 5450 50  0000 C CNN
 	1    3750 5450
