File: V2/design_files_2-1/base.kicad_pcb (KiCad board)
At the start: 2 copper layers, 31.8 x 58.4 mm, 35 parts, among them J1 Isty_Left, J2 Itsy_right, P3 LEFT_STEPPER, P4 RIGHT_STEPPER, P5 BATT1, P6 BATT2, P7 SERVO, P9 CONN_01X01, Q1 OPTO_NPN, Q2 OPTO_NPN, Q3 2N4401, SW1 SPST, SW2 SW_PUSH, U1 ULN2803

Commit message: Updates
Parts:
- removed Q3: 2N4401, TO_SOT_Packages_THT:TO-92_Inline_Wide
- removed R10: 10K, library:Resistor_Horz
- removed R9: 1000, library:Resistor_Horz
- R2, R5: value 47 -> 330
- turned R1 to 0 degrees
Connections:
- J2 pad 12: /A2 -> /SDA
- P7 pad 1: /D5 -> /A1
- Q1 pad 3: /A2 -> /A3
- Q2 pad 3: /A1 -> /A2
- R1 pad 1: /A2 -> /SDA
- R1 pad 2: /A2 -> /A3
- R2 pad 1: Net-(Q3-Pad1) -> /D5
- R5 pad 1: Net-(Q3-Pad1) -> /D5
- R6 pad 2: /A1 -> /A2
- R7 pad 2: /A2 -> /A3
- R8 pad 2: /A1 -> /A2
- U1 pad 2: /A3 -> /D10
Routing:
- net /A2: track 125.0 -> 35.7 mm
- net /A3: track 2.54 -> 75.2 mm
- net /SDA: track 0.00 -> 52.4 mm
- net /A1: track 34.3 -> 62.5 mm
- net /D5: track 25.9 -> 45.7 mm
- net GND: track 175.5 -> 160.3 mm
- net /D10: track 0.00 -> 13.8 mm
- net /D7: track 33.4 -> 41.3 mm
- net /D11: track 42.6 -> 46.7 mm
- net Net-(Q3-Pad1): track 1.53 -> 0.00 mm
- net /D12: track 31.7 -> 33.0 mm
- net /SCL: track 13.2 -> 12.0 mm
- net /A0: track 0.89 -> 0.13 mm
Other:
- board text added: "A2"
- board text added: "A3"
- board text added: "D5"
- board text added: "SERVO"
- board text added: "SWITCH"
- board text added: "Ver 2.1 Nov 2019"
- board text removed: "A0"
- board text removed: "A1"
- board text removed: "D10"
- board text removed: "D13"
- board text removed: "Ver 0.5 Aug 2018"

Commit message: Updates
Parts:
- added LS1: Speaker, library:PS1240_piezo, F.Cu at (139.8, 67.9)
Routing:
- net /A0: track 0.13 -> 111.1 mm, vias 0 -> 1
- net /A1: track 62.5 -> 61.6 mm
- net /A2: track 35.7 -> 35.1 mm

Commit message: Updates
Parts:
- D3, D4: footprint LEDs:LED-3MM -> library:LED-3MM_RA
- J1: footprint Pin_Headers:Pin_Header_Straight_1x14_Pitch2.54mm -> library:Pin_Header_Straight_1x14_Pitch2.54mm
- J2: footprint Pin_Headers:Pin_Header_Straight_1x14_Pitch2.54mm -> Pin_Header_Straight_1x14_Pitch2.54mm
- P3: footprint library:JST_B5B-XH-A -> JST_B5B-XH-A
- Q1: footprint library:PHOTOTRANS-RA -> PHOTOTRANS-RA
- Q2: footprint myFootPrints:PHOTOTRANS -> library:PHOTOTRANS-RA
- R2, R3, R4, R5, R6, R7: footprint myFootPrints:Resistor_Horz -> library:Resistor_Horz
- moved R8 6.86 mm to (132.3, 94.0)
- moved R2 2.54 mm to (151.1, 97.8)
- moved R3 2.54 mm to (148.6, 80.0)
- moved R4 2.54 mm to (148.6, 97.8)
- moved R5 2.54 mm to (151.1, 80.0)
- moved LS1 2.03 mm to (141.9, 67.9)
- moved C3 0.63 mm to (132.7, 111.1)
- moved D2 0.63 mm to (148.0, 111.1)
- moved D3 0.63 mm to (148.0, 74.3)
- moved D4 0.63 mm to (148.0, 106.0)
- moved D5 0.63 mm to (148.0, 69.2)
- moved Q1 0.63 mm to (148.0, 62.9)
- moved Q2 0.63 mm to (148.0, 114.9)
Routing:
- net GND: track 160.0 -> 186.1 mm
- net /A2: track 35.1 -> 49.4 mm
- net Net-(D5-Pad2): track 20.7 -> 12.3 mm
- net Net-(D4-Pad2): track 11.2 -> 3.31 mm
- net /SCL: track 12.0 -> 5.11 mm
- net /A0: track 111.1 -> 104.5 mm
- net /D7: track 41.3 -> 34.8 mm
- net /D11: track 46.7 -> 41.1 mm
- net /A3: track 75.3 -> 70.0 mm
- net /D5: track 45.7 -> 48.3 mm
- net Net-(P3-Pad4): track 18.8 -> 19.7 mm
Other:
- board text added: "NPN"
- board text added: "Ver 2.2 Feb 2020"
- board text removed: "Ver 2.1 Nov 2019"

Commit message: Updates
Other:
- board text added: "JLCJLCJLCJLC"
Changed lines of the file:
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@@
     (area 121.792999 59.562999 153.797001 118.237001)
     (thickness 1.6)
-    (drawings 53)
+    (drawings 54)
     (tracks 354)
     (zones 0)
@@
   )
   (setup
-    (last_trace_width 0.6096)
+    (last_trace_width 0.1524)
     (user_trace_width 0.254)
     (user_trace_width 0.3048)
@@
     )
   )
+  (gr_text JLCJLCJLCJLC (at 152.019 109.855 90) (layer B.SilkS)
+    (effects (font (size 1 1) (thickness 0.25)) (justify mirror))
+  )
   (gr_text NPN (at 151.003 115.062) (layer F.SilkS)
     (effects (font (size 1.016 1.016) (thickness 0.254)))
@@
     (effects (font (size 1.016 1.016) (thickness 0.254)))
   )
-  (gr_text SWITCH (at 134.747 64.135) (layer B.SilkS)
+  (gr_text SWITCH (at 134.747 64.389) (layer B.SilkS)
     (effects (font (size 1.5 1.5) (thickness 0.3)) (justify mirror))
   )

Commit message: Updates
Parts:
- removed R1, R8: 0, Resistors_SMD:R_0402
- Q1: footprint PHOTOTRANS-RA -> library:PHOTOTRANS-RA
- moved C3 2.67 mm to (132.7, 113.8), turned to 90 degrees
- moved C2 2.25 mm to (134.9, 105.0), turned to 270 degrees
- moved LS1 0.74 mm to (142.2, 68.6)
- moved P7 0.63 mm to (134.6, 75.6)
Routing:
- net /SDA: track 52.4 -> 0.00 mm
- net /A2: track 49.4 -> 24.5 mm
- net /A3: track 70.0 -> 58.3 mm
- net GND: track 186.1 -> 180.4 mm
- net /BAT: track 90.7 -> 96.2 mm
- net /SCL: track 5.11 -> 1.02 mm
- net /A0: track 104.5 -> 105.2 mm
