File: V2/design_files_2-1/base.sch (KiCad schematic (older format))
At the start: 30 parts, among them J1 Isty_Left, J2 Itsy_right, P3 LEFT_STEPPER, P4 RIGHT_STEPPER, P5 BATT1, P6 BATT2, P7 SERVO, Q1 OPTO_NPN, Q2 OPTO_NPN, Q3 2N4401, SW1 SPST, SW2 SW_PUSH, U1 ULN2803

Commit message: Updates
Parts:
- removed Q3: 2N4401, TO_SOT_Packages_THT:TO-92_Inline_Wide, symbol Q_NPN_EBC
- removed R10: 10K, library:Resistor_Horz, symbol R
- removed R9: 1000, library:Resistor_Horz, symbol R
- R2, R5: value 47 -> 330
Connections:
- wire segments 93 -> 88
Other:
- note added: "IR 1.2Vf 330 ohm 12 mA @ 5V"
Changed lines of the file:
@@
 P 6250 5600
 F 0 "R2" V 6330 5600 50  0000 C CNN
-F 1 "47" V 6250 5600 50  0000 C CNN
+F 1 "330" V 6250 5600 50  0000 C CNN
 F 2 "library:Resistor_Horz" V 6180 5600 50  0001 C CNN
 F 3 "" H 6250 5600 50  0000 C CNN
@@
 P 5350 5600
 F 0 "R5" V 5430 5600 50  0000 C CNN
-F 1 "47" V 5350 5600 50  0000 C CNN
+F 1 "330" V 5350 5600 50  0000 C CNN
 F 2 "library:Resistor_Horz" V 5280 5600 50  0001 C CNN
 F 3 "" H 5350 5600 50  0000 C CNN
@@
 Text Label 5850 3350 0    60   ~ 0
 A4
-Text Label 5850 3250 0    60   ~ 0
+Text Label 3850 5250 0    60   ~ 0
 A3
 Text Label 5850 3150 0    60   ~ 0
@@
 Text Label 5850 3850 0    60   ~ 0
 D9
+Text Label 6950 2500 0    60   ~ 0
+A1
 Text Label 3850 4750 0    60   ~ 0
-A1
-Text Label 3850 5250 0    60   ~ 0
 A2
 Text Label 3850 5050 0    60   ~ 0
 D7
-Text Label 2500 5300 0    60   ~ 0
+Text Label 5850 3250 0    60   ~ 0
 D10
 Text Label 3850 4950 0    60   ~ 0
@@
 Text Label 3850 5350 0    60   ~ 0
 D12
-Text Label 6950 2500 0    60   ~ 0
+Text Label 3300 4900 0    60   ~ 0
 D5
 NoConn ~ 2850 2800
@@
 	4600 5350 3850 5350
 Wire Wire Line
-	4800 3800 4800 4500
+	4800 3800 4800 4250
 Connection ~ 4600 4250
 Connection ~ 4600 4550
 Connection ~ 4800 4250
 Connection ~ 4800 4550
-$Comp
-L Q_NPN_EBC Q3
-U 1 1 5DB780E7
-P 3200 5000
-F 0 "Q3" H 3400 5050 50  0000 L CNN
-F 1 "2N4401" H 3400 4950 50  0000 L CNN
-F 2 "TO_SOT_Packages_THT:TO-92_Inline_Wide" H 3400 5100 50  0001 C CNN
-F 3 "" H 3200 5000 50  0001 C CNN
-	1    3200 5000
-	0    -1   -1   0
-$EndComp
 Wire Wire Line
 	3550 4850 3550 5150
 Wire Wire Line
-	3550 4900 3400 4900
+	3550 4900 3300 4900
 Connection ~ 3550 4900
-$Comp
-L R R9
-U 1 1 5DB78348
-P 2900 5300
-F 0 "R9" V 2980 5300 50  0000 C CNN
-F 1 "1000" V 2900 5300 50  0000 C CNN
-F 2 "library:Resistor_Horz" V 2830 5300 50  0001 C CNN
-F 3 "" H 2900 5300 50  0000 C CNN
-	1    2900 5300
-	0    1    1    0
-$EndComp
-Wire Wire Line
-	2500 5300 2750 5300
-$Comp
-L R R10
-U 1 1 5DB7854E
-P 3200 5550
-F 0 "R10" V 3280 5550 50  0000 C CNN
-F 1 "10K" V 3200 5550 50  0000 C CNN
-F 2 "library:Resistor_Horz" V 3130 5550 50  0001 C CNN
-F 3 "" H 3200 5550 50  0000 C CNN
-	1    3200 5550
-	-1   0    0    1
-$EndComp
-$Comp
-L GND #PWR016
-U 1 1 5DB785DC
-P 3200 5800
-F 0 "#PWR016" H 3200 5550 50  0001 C CNN
-F 1 "GND" H 3200 5650 50  0000 C CNN
-F 2 "" H 3200 5800 60  0000 C CNN
-F 3 "" H 3200 5800 60  0000 C CNN
-	1    3200 5800
-	1    0    0    -1
-$EndComp
-$Comp
-L +3.3V #PWR017
-U 1 1 5DB786A0
-P 2800 4800
-F 0 "#PWR017" H 2800 4650 50  0001 C CNN
-F 1 "+3.3V" H 2800 4940 50  0000 C CNN
-F 2 "" H 2800 4800 50  0001 C CNN
-F 3 "" H 2800 4800 50  0001 C CNN
-	1    2800 4800
-	1    0    0    -1
-$EndComp
-Wire Wire Line
-	2800 4800 2800 4900
-Wire Wire Line
-	2800 4900 3000 4900
-Wire Wire Line
-	3050 5300 3200 5300
-Wire Wire Line
-	3200 5200 3200 5400
-Connection ~ 3200 5300
-Wire Wire Line
-	3200 5700 3200 5800
-Wire Wire Line
-	4600 3900 4600 5250
 Connection ~ 4600 5250
 Wire Wire Line
 	4800 4550 4800 4750
 Connection ~ 4800 4750
+Wire Wire Line
+	4600 3900 4600 4250
+Wire Wire Line
+	4600 4550 4600 5250
+Text Notes 7100 5300 0    60   ~ 0
+IR 1.2Vf 330 ohm 12 mA @ 5V
 $EndSCHEMATC

Commit message: Updates
Parts:
- added LS1: Speaker, library:PS1240_piezo, symbol Speaker
Connections:
- wire segments 88 -> 90
Other:
- moved on the sheet: SW2
Changed lines of the file:
@@
 $EndDescr
 $Comp
-L PWR_FLAG #FLG01
+L PWR_FLAG #FLG1
 U 1 1 553FAE81
 P 900 900
-F 0 "#FLG01" H 900 995 50  0001 C CNN
+F 0 "#FLG1" H 900 995 50  0001 C CNN
 F 1 "PWR_FLAG" H 900 1080 50  0000 C CNN
 F 2 "" H 900 900 60  0000 C CNN
@@
 $EndComp
 $Comp
-L PWR_FLAG #FLG02
+L PWR_FLAG #FLG3
 U 1 1 553FAEA5
 P 1550 900
-F 0 "#FLG02" H 1550 995 50  0001 C CNN
+F 0 "#FLG3" H 1550 995 50  0001 C CNN
 F 1 "PWR_FLAG" H 1550 1080 50  0000 C CNN
 F 2 "" H 1550 900 60  0000 C CNN
@@
 $EndComp
 $Comp
-L GND #PWR03
+L GND #PWR3
 U 1 1 553FAEE7
 P 1550 1000
-F 0 "#PWR03" H 1550 750 50  0001 C CNN
+F 0 "#PWR3" H 1550 750 50  0001 C CNN
 F 1 "GND" H 1550 850 50  0000 C CNN
 F 2 "" H 1550 1000 60  0000 C CNN
@@
 $EndComp
 $Comp
-L +BATT #PWR04
+L +BATT #PWR1
 U 1 1 553FAF12
 P 900 1000
-F 0 "#PWR04" H 900 850 50  0001 C CNN
+F 0 "#PWR1" H 900 850 50  0001 C CNN
 F 1 "+BATT" H 900 1140 50  0000 C CNN
 F 2 "" H 900 1000 60  0000 C CNN
@@
 $EndComp
 $Comp
-L GND #PWR05
+L GND #PWR12
 U 1 1 59BB5846
 P 6550 4000
-F 0 "#PWR05" H 6550 3750 50  0001 C CNN
+F 0 "#PWR12" H 6550 3750 50  0001 C CNN
 F 1 "GND" H 6550 3850 50  0000 C CNN
 F 2 "" H 6550 4000 60  0000 C CNN
@@
 $EndComp
 $Comp
-L GND #PWR06
+L GND #PWR13
 U 1 1 59BB84D9
 P 7350 2350
-F 0 "#PWR06" H 7350 2100 50  0001 C CNN
+F 0 "#PWR13" H 7350 2100 50  0001 C CNN
 F 1 "GND" H 7350 2200 50  0000 C CNN
 F 2 "" H 7350 2350 60  0000 C CNN
@@
 $EndComp
 $Comp
-L GND #PWR07
+L GND #PWR10
 U 1 1 59BB875A
 P 5400 3100
-F 0 "#PWR07" H 5400 2850 50  0001 C CNN
+F 0 "#PWR10" H 5400 2850 50  0001 C CNN
 F 1 "GND" H 5400 2950 50  0000 C CNN
 F 2 "" H 5400 3100 60  0000 C CNN
@@
 $EndComp
 $Comp
-L GND #PWR08
+L GND #PWR6
 U 1 1 59BB9EFB
-P 4600 6050
-F 0 "#PWR08" H 4600 5800 50  0001 C CNN
-F 1 "GND" H 4600 5900 50  0000 C CNN
-F 2 "" H 4600 6050 60  0000 C CNN
-F 3 "" H 4600 6050 60  0000 C CNN
-	1    4600 6050
-	1    0    0    -1
-$EndComp
-$Comp
-L GND #PWR09
+P 4600 6100
+F 0 "#PWR6" H 4600 5850 50  0001 C CNN
+F 1 "GND" H 4600 5950 50  0000 C CNN
+F 2 "" H 4600 6100 60  0000 C CNN
+F 3 "" H 4600 6100 60  0000 C CNN
+	1    4600 6100
+	1    0    0    -1
+$EndComp
+$Comp
+L GND #PWR7
 U 1 1 59CB1B18
 P 4750 2050
-F 0 "#PWR09" H 4750 1800 50  0001 C CNN
+F 0 "#PWR7" H 4750 1800 50  0001 C CNN
 F 1 "GND" H 4750 1900 50  0000 C CNN
 F 2 "" H 4750 2050 60  0000 C CNN
@@
 $EndComp
 $Comp
-L GND #PWR010
+L GND #PWR9
 U 1 1 59FA7C9A
 P 5350 6150
-F 0 "#PWR010" H 5350 5900 50  0001 C CNN
+F 0 "#PWR9" H 5350 5900 50  0001 C CNN
 F 1 "GND" H 5350 6000 50  0000 C CNN
 F 2 "" H 5350 6150 60  0000 C CNN
@@
 $EndComp
 $Comp
-L GND #PWR011
+L GND #PWR11
 U 1 1 59FA7CFD
 P 6250 6150
-F 0 "#PWR011" H 6250 5900 50  0001 C CNN
+F 0 "#PWR11" H 6250 5900 50  0001 C CNN
 F 1 "GND" H 6250 6000 50  0000 C CNN
 F 2 "" H 6250 6150 60  0000 C CNN
@@
 L SW_PUSH SW2
 U 1 1 59FBD881
-P 4600 5750
-F 0 "SW2" H 4750 5860 50  0000 C CNN
-F 1 "SW_PUSH" H 4600 5670 50  0000 C CNN
-F 2 "library:SW_PUSH_SMALL" H 4600 5750 50  0001 C CNN
-F 3 "" H 4600 5750 50  0000 C CNN
-	1    4600 5750
+P 4600 5800
+F 0 "SW2" H 4750 5910 50  0000 C CNN
+F 1 "SW_PUSH" H 4600 5720 50  0000 C CNN
+F 2 "library:SW_PUSH_SMALL" H 4600 5800 50  0001 C CNN
+F 3 "" H 4600 5800 50  0000 C CNN
+	1    4600 5800
 	0    1    1    0
 $EndComp
@@
 RX
 $Comp
-L PWR_FLAG #FLG012
+L PWR_FLAG #FLG2
 U 1 1 5ADA8A03
 P 1200 900
-F 0 "#FLG012" H 1200 995 50  0001 C CNN
+F 0 "#FLG2" H 1200 995 50  0001 C CNN
 F 1 "PWR_FLAG" H 1200 1080 50  0000 C CNN
 F 2 "" H 1200 900 60  0000 C CNN
@@
 $EndComp
 $Comp
-L +3.3V #PWR013
+L +3.3V #PWR2
 U 1 1 5ADA8A47
 P 1200 1000
-F 0 "#PWR013" H 1200 850 50  0001 C CNN
+F 0 "#PWR2" H 1200 850 50  0001 C CNN
 F 1 "+3.3V" H 1200 1140 50  0000 C CNN
 F 2 "" H 1200 1000 50  0001 C CNN
@@
 $EndComp
 $Comp
-L +3.3V #PWR014
+L +3.3V #PWR4
 U 1 1 5ADA90E0
 P 2850 2900
-F 0 "#PWR014" H 2850 2750 50  0001 C CNN
+F 0 "#PWR4" H 2850 2750 50  0001 C CNN
 F 1 "+3.3V" H 2850 3040 50  0000 C CNN
 F 2 "" H 2850 2900 50  0001 C CNN
@@
 $EndComp
 $Comp
-L +3.3V #PWR015
+L +3.3V #PWR8
 U 1 1 5ADA9793
 P 5350 4050
-F 0 "#PWR015" H 5350 3900 50  0001 C CNN
+F 0 "#PWR8" H 5350 3900 50  0001 C CNN
 F 1 "+3.3V" H 5350 4190 50  0000 C CNN
 F 2 "" H 5350 4050 50  0001 C CNN
@@
 	5500 4550 5500 4750
 Wire Wire Line
-	4600 5450 4600 5350
+	4600 5350 4600 5500
 Wire Wire Line
 	4600 5350 3850 5350
@@
 Text Notes 7100 5300 0    60   ~ 0
 IR 1.2Vf 330 ohm 12 mA @ 5V
+$Comp
+L Speaker LS1
+U 1 1 5DE2C66A
+P 4250 5700
+F 0 "LS1" H 4300 5925 50  0000 R CNN
+F 1 "Speaker" H 4300 5850 50  0000 R CNN
+F 2 "library:PS1240_piezo" H 4250 5500 50  0001 C CNN
+F 3 "" H 4240 5650 50  0001 C CNN
+	1    4250 5700
+	1    0    0    -1
+$EndComp
+Wire Wire Line
+	4050 5700 3850 5700
+$Comp
+L GND #PWR5
+U 1 1 5DE2C798
+P 4050 6100
+F 0 "#PWR5" H 4050 5850 50  0001 C CNN
+F 1 "GND" H 4050 5950 50  0000 C CNN
+F 2 "" H 4050 6100 60  0000 C CNN
+F 3 "" H 4050 6100 60  0000 C CNN
+	1    4050 6100
+	1    0    0    -1
+$EndComp
+Wire Wire Line
+	4050 5800 4050 6100
+Text Label 3850 5700 0    60   ~ 0
+A0
 $EndSCHEMATC

Commit message: Updates
Parts:
- removed R1, R8: 0, library:R_0402, symbol R
Connections:
- wire segments 90 -> 86
- no-connect marks 7 -> 9
Changed lines of the file:
@@
 $EndDescr
 $Comp
-L PWR_FLAG #FLG1
+L PWR_FLAG #FLG01
 U 1 1 553FAE81
 P 900 900
-F 0 "#FLG1" H 900 995 50  0001 C CNN
+F 0 "#FLG01" H 900 995 50  0001 C CNN
 F 1 "PWR_FLAG" H 900 1080 50  0000 C CNN
 F 2 "" H 900 900 60  0000 C CNN
@@
 $EndComp
 $Comp
-L PWR_FLAG #FLG3
+L PWR_FLAG #FLG02
 U 1 1 553FAEA5
 P 1550 900
-F 0 "#FLG3" H 1550 995 50  0001 C CNN
+F 0 "#FLG02" H 1550 995 50  0001 C CNN
 F 1 "PWR_FLAG" H 1550 1080 50  0000 C CNN
 F 2 "" H 1550 900 60  0000 C CNN
@@
 $EndComp
 $Comp
-L GND #PWR3
+L GND #PWR03
 U 1 1 553FAEE7
 P 1550 1000
-F 0 "#PWR3" H 1550 750 50  0001 C CNN
+F 0 "#PWR03" H 1550 750 50  0001 C CNN
 F 1 "GND" H 1550 850 50  0000 C CNN
 F 2 "" H 1550 1000 60  0000 C CNN
@@
 $EndComp
 $Comp
-L +BATT #PWR1
+L +BATT #PWR04
 U 1 1 553FAF12
 P 900 1000
-F 0 "#PWR1" H 900 850 50  0001 C CNN
+F 0 "#PWR04" H 900 850 50  0001 C CNN
 F 1 "+BATT" H 900 1140 50  0000 C CNN
 F 2 "" H 900 1000 60  0000 C CNN
@@
 $EndComp
 $Comp
-L GND #PWR12
+L GND #PWR05
 U 1 1 59BB5846
 P 6550 4000
-F 0 "#PWR12" H 6550 3750 50  0001 C CNN
+F 0 "#PWR05" H 6550 3750 50  0001 C CNN
 F 1 "GND" H 6550 3850 50  0000 C CNN
 F 2 "" H 6550 4000 60  0000 C CNN
@@
 $EndComp
 $Comp
-L GND #PWR13
+L GND #PWR06
 U 1 1 59BB84D9
 P 7350 2350
-F 0 "#PWR13" H 7350 2100 50  0001 C CNN
+F 0 "#PWR06" H 7350 2100 50  0001 C CNN
 F 1 "GND" H 7350 2200 50  0000 C CNN
 F 2 "" H 7350 2350 60  0000 C CNN
@@
 $EndComp
 $Comp
-L GND #PWR10
+L GND #PWR07
 U 1 1 59BB875A
 P 5400 3100
-F 0 "#PWR10" H 5400 2850 50  0001 C CNN
+F 0 "#PWR07" H 5400 2850 50  0001 C CNN
 F 1 "GND" H 5400 2950 50  0000 C CNN
 F 2 "" H 5400 3100 60  0000 C CNN
@@
 $EndComp
 $Comp
-L GND #PWR6
+L GND #PWR08
 U 1 1 59BB9EFB
 P 4600 6100
-F 0 "#PWR6" H 4600 5850 50  0001 C CNN
+F 0 "#PWR08" H 4600 5850 50  0001 C CNN
 F 1 "GND" H 4600 5950 50  0000 C CNN
 F 2 "" H 4600 6100 60  0000 C CNN
@@
 $EndComp
 $Comp
-L GND #PWR7
+L GND #PWR09
 U 1 1 59CB1B18
 P 4750 2050
-F 0 "#PWR7" H 4750 1800 50  0001 C CNN
+F 0 "#PWR09" H 4750 1800 50  0001 C CNN
 F 1 "GND" H 4750 1900 50  0000 C CNN
 F 2 "" H 4750 2050 60  0000 C CNN
@@
 $EndComp
 $Comp
-L GND #PWR9
+L GND #PWR010
 U 1 1 59FA7C9A
 P 5350 6150
-F 0 "#PWR9" H 5350 5900 50  0001 C CNN
+F 0 "#PWR010" H 5350 5900 50  0001 C CNN
 F 1 "GND" H 5350 6000 50  0000 C CNN
 F 2 "" H 5350 6150 60  0000 C CNN
@@
 $EndComp
 $Comp
-L GND #PWR11
+L GND #PWR011
 U 1 1 59FA7CFD
 P 6250 6150
-F 0 "#PWR11" H 6250 5900 50  0001 C CNN
+F 0 "#PWR011" H 6250 5900 50  0001 C CNN
 F 1 "GND" H 6250 6000 50  0000 C CNN
 F 2 "" H 6250 6150 60  0000 C CNN
@@
 RX
 $Comp
-L PWR_FLAG #FLG2
+L PWR_FLAG #FLG012
 U 1 1 5ADA8A03
 P 1200 900
-F 0 "#FLG2" H 1200 995 50  0001 C CNN
+F 0 "#FLG012" H 1200 995 50  0001 C CNN
 F 1 "PWR_FLAG" H 1200 1080 50  0000 C CNN
 F 2 "" H 1200 900 60  0000 C CNN
@@
 $EndComp
 $Comp
-L +3.3V #PWR2
+L +3.3V #PWR013
 U 1 1 5ADA8A47
 P 1200 1000
-F 0 "#PWR2" H 1200 850 50  0001 C CNN
+F 0 "#PWR013" H 1200 850 50  0001 C CNN
 F 1 "+3.3V" H 1200 1140 50  0000 C CNN
 F 2 "" H 1200 1000 50  0001 C CNN
@@
 $EndComp
 $Comp
-L +3.3V #PWR4
+L +3.3V #PWR014
 U 1 1 5ADA90E0
 P 2850 2900
-F 0 "#PWR4" H 2850 2750 50  0001 C CNN
+F 0 "#PWR014" H 2850 2750 50  0001 C CNN
 F 1 "+3.3V" H 2850 3040 50  0000 C CNN
 F 2 "" H 2850 2900 50  0001 C CNN
@@
 $EndComp
 $Comp
-L +3.3V #PWR8
+L +3.3V #PWR015
 U 1 1 5ADA9793
 P 5350 4050
-F 0 "#PWR8" H 5350 3900 50  0001 C CNN
+F 0 "#PWR015" H 5350 3900 50  0001 C CNN
 F 1 "+3.3V" H 5350 4190 50  0000 C CNN
 F 2 "" H 5350 4050 50  0001 C CNN
@@
 NoConn ~ 4150 4000
 NoConn ~ 4150 4100
-$Comp
-L R R1
-U 1 1 5B3AEB76
-P 4600 4400
-F 0 "R1" V 4680 4400 50  0000 C CNN
-F 1 "0" V 4600 4400 50  0000 C CNN
-F 2 "library:R_0402" V 4530 4400 50  0001 C CNN
-F 3 "" H 4600 4400 50  0000 C CNN
-	1    4600 4400
-	1    0    0    -1
-$EndComp
-$Comp
-L R R8
-U 1 1 5B3AEBE4
-P 4800 4400
-F 0 "R8" V 4880 4400 50  0000 C CNN
-F 1 "0" V 4800 4400 50  0000 C CNN
-F 2 "library:R_0402" V 4730 4400 50  0001 C CNN
-F 3 "" H 4800 4400 50  0000 C CNN
-	1    4800 4400
-	1    0    0    -1
-$EndComp
 Wire Wire Line
 	900  900  900  1000
@@
 	4050 3700 4150 3700
 Wire Wire Line
-	4050 3800 4800 3800
-Wire Wire Line
-	4050 3900 4600 3900
-Wire Wire Line
 	4050 4000 4150 4000
 Wire Wire Line
@@
 	4600 5350 3850 5350
 Wire Wire Line
-	4800 3800 4800 4250
-Connection ~ 4600 4250
-Connection ~ 4600 4550
-Connection ~ 4800 4250
-Connection ~ 4800 4550
-Wire Wire Line
 	3550 4850 3550 5150
 Wire Wire Line
 	3550 4900 3300 4900
 Connection ~ 3550 4900
-Connection ~ 4600 5250
-Wire Wire Line
-	4800 4550 4800 4750
-Connection ~ 4800 4750
-Wire Wire Line
-	4600 3900 4600 4250
-Wire Wire Line
-	4600 4550 4600 5250
 Text Notes 7100 5300 0    60   ~ 0
 IR 1.2Vf 330 ohm 12 mA @ 5V
@@
 	4050 5700 3850 5700
 $Comp
-L GND #PWR5
+L GND #PWR016
 U 1 1 5DE2C798
 P 4050 6100
-F 0 "#PWR5" H 4050 5850 50  0001 C CNN
+F 0 "#PWR016" H 4050 5850 50  0001 C CNN
 F 1 "GND" H 4050 5950 50  0000 C CNN
 F 2 "" H 4050 6100 60  0000 C CNN
@@
 Text Label 3850 5700 0    60   ~ 0
 A0
+NoConn ~ 4150 3800
+NoConn ~ 4150 3900
+Wire Wire Line
+	4050 3800 4150 3800
+Wire Wire Line
+	4050 3900 4150 3900
 $EndSCHEMATC
